Commit message: Update the xacro files to work in ROS2

File: unitree_a1_desc/xacro/const.xacro (robot description, xacro)
@@ -1,4 +1,4 @@
 <?xml version="1.0"?>
-<robot name="a1_description" xmlns:xacro="http://www.ros.org/wiki/xacro">
+<robot name="unitree_a1_desc" xmlns:xacro="http://www.ros.org/wiki/xacro">
     <!-- Constants for robot dimensions -->
     <xacro:property name="PI" value="3.1415926535897931"/>

File: unitree_a1_desc/xacro/leg.xacro (robot description, xacro)
@@ -1,5 +1,5 @@
 <?xml version="1.0"?>
 <robot xmlns:xacro="http://www.ros.org/wiki/xacro">
-    <xacro:include filename="$(find a1_description)/xacro/transmission.xacro"/>
+    <xacro:include filename="$(find unitree_a1_desc)/transmission.xacro"/>
     <xacro:macro name="leg" params="name mirror mirror_dae front_hind front_hind_dae *origin">
         <joint name="${name}_hip_joint" type="revolute">
@@ -31,5 +31,5 @@
                 </xacro:if>
                 <geometry>
-                    <mesh filename="package://a1_description/meshes/hip.dae" scale="1 1 1"/>
+                    <mesh filename="package://unitree_a1_desc/meshes/hip.dae" scale="1 1 1"/>
                 </geometry>
                 <material name="orange"/>
@@ -77,8 +77,8 @@
                 <geometry>
                     <xacro:if value="${mirror_dae == True}">
-                        <mesh filename="package://a1_description/meshes/thigh.dae" scale="1 1 1"/>
+                        <mesh filename="package://unitree_a1_desc/meshes/thigh.dae" scale="1 1 1"/>
                     </xacro:if>
                     <xacro:if value="${mirror_dae == False}">
-                        <mesh filename="package://a1_description/meshes/thigh_mirror.dae" scale="1 1 1"/>
+                        <mesh filename="package://unitree_a1_desc/meshes/thigh_mirror.dae" scale="1 1 1"/>
                     </xacro:if>
                 </geometry>
@@ -112,5 +112,5 @@
                 <origin rpy="0 0 0" xyz="0 0 0"/>
                 <geometry>
-                    <mesh filename="package://a1_description/meshes/calf.dae" scale="1 1 1"/>
+                    <mesh filename="package://unitree_a1_desc/meshes/calf.dae" scale="1 1 1"/>
                 </geometry>
                 <material name="orange"/>

File: unitree_a1_desc/xacro/robot.xacro (robot description, xacro)
@@ -1,8 +1,8 @@
 <?xml version="1.0"?>
-<robot name="a1_description" xmlns:xacro="http://www.ros.org/wiki/xacro">
-    <xacro:include filename="$(find a1_description)/xacro/const.xacro"/>
-    <xacro:include filename="$(find a1_description)/xacro/materials.xacro"/>
-    <xacro:include filename="$(find a1_description)/xacro/leg.xacro"/>
-    <xacro:include filename="$(find a1_description)/xacro/stairs.xacro"/>
+<robot name="unitree_a1_desc" xmlns:xacro="http://www.ros.org/wiki/xacro">
+    <xacro:include filename="$(find unitree_a1_desc)/const.xacro"/>
+    <xacro:include filename="$(find unitree_a1_desc)/materials.xacro"/>
+    <xacro:include filename="$(find unitree_a1_desc)/leg.xacro"/>
+    <xacro:include filename="$(find unitree_a1_desc)/stairs.xacro"/>
     <!-- <xacro:include filename="$(find a1_gazebo)/launch/gazebo.xacro"/> -->
     <!-- <xacro:include filename="$(find a1_gazebo)/launch/stairs.urdf.xacro"/> -->
@@ -11,5 +11,5 @@
     <xacro:property name="rolloverProtection" value="false"/>
     <!-- Debug mode will hung up the robot, use "true" or "false" to switch it. -->
-    <xacro:if value="$(arg DEBUG)">
+<!--    <xacro:if value="$(arg DEBUG)">
         <link name="world"/>
         <joint name="base_static_joint" type="fixed">
@@ -19,4 +19,5 @@
         </joint>
     </xacro:if>
+-->
     <link name="base">
         <visual>
@@ -36,5 +37,5 @@
             <origin rpy="0 0 0" xyz="0 0 0"/>
             <geometry>
-                <mesh filename="package://a1_description/meshes/trunk.dae" scale="1 1 1"/>
+                <mesh filename="package://unitree_a1_desc/meshes/trunk.dae" scale="1 1 1"/>
             </geometry>
             <material name="orange"/>
